Commit message: calibration fixs. thread fixes, cleanup , urdf cleanup

File: urdf/stereo_camera.urdf.xacro (robot description, xacro)
@@ -7,5 +7,5 @@
   <xacro:macro name="stereo_camera_macro" params="parent *origin">
     <!-- Base link -->
-    <link name="stereo_camera_base">
+    <link name="camera_link">
       <visual>
         <geometry>
@@ -25,5 +25,5 @@
     <link name="left_camera_frame"/>
     <joint name="left_camera_joint" type="fixed">
-      <parent link="stereo_camera_base"/>
+      <parent link="camera_link"/>
       <child link="left_camera_frame"/>
       <origin xyz="${-baseline/2} 0 0" rpy="0 0 0"/>
@@ -32,5 +32,5 @@
     <link name="right_camera_frame"/>
     <joint name="right_camera_joint" type="fixed">
-      <parent link="stereo_camera_base"/>
+      <parent link="camera_link"/>
       <child link="right_camera_frame"/>
       <origin xyz="${baseline/2} 0 0" rpy="0 0 0"/>
@@ -39,5 +39,5 @@
     <link name="imu_link"/>
     <joint name="imu_joint" type="fixed">
-      <parent link="stereo_camera_base"/>
+      <parent link="camera_link"/>
       <child link="imu_link"/>
       <origin xyz="0 0 0" rpy="0 0 0"/>
@@ -47,11 +47,11 @@
       <xacro:insert_block name="origin"/>
       <parent link="${parent}"/>
-      <child link="stereo_camera_base"/>
+      <child link="camera_link"/>
     </joint>
   </xacro:macro>
-  <!-- Create world link if needed -->
-  <link name="world"/>
+  <!-- Create base link -->
+  <link name="base_link"/>
   <!-- Instantiate the stereo camera -->
-  <xacro:stereo_camera_macro parent="world">
+  <xacro:stereo_camera_macro parent="base_link">
     <origin xyz="0 0 0" rpy="0 0 0"/>
   </xacro:stereo_camera_macro>
